File: Power-Interposer-Board-AC/Power-Interposer-Board-AC.kicad_pcb (KiCad board)
At the start: 2 copper layers, 71.1 x 40.6 mm, 7 parts, among them J1 AC_Pwr_IN, J2 AC_Pwr_OUT, J3 AC_Sense

Commit message: Minor Updates
Parts:
- removed J3: AC_Sense, Connector_JST:JST_VH_B2P-VH_1x02_P3.96mm_Vertical
- added BJ1: Sense_OUT, Connector:CalTest_CT3151, F.Cu at (162.6, 106.7)
- added BJ2: Sense_IN, Connector:CalTest_CT3151, F.Cu at (162.6, 126.7)
- moved J1 0.15 mm to (127.0, 110.3)
Routing:
- net Net-(BJ2-Pad1): track 13.7 -> 52.2 mm
- net Net-(BJ1-Pad1): track 20.0 -> 47.4 mm
- net Net-(J1-Pad1): vias 6 -> 5
