File: Battery-Holders/Battery-Holders.sch (KiCad schematic (older format))
At the start: 12 parts, among them J1 Conn_01x02

Commit message: Minor Updates
Parts:
- removed BT3, BT4, BT5: Battery, Battery:BatteryHolder_MPD_BH-18650-PC2, symbol Device:Battery
- removed D1: D, Package_TO_SOT_THT:TO-247-2_Horizontal_TabDown, symbol Device:D
- added D1: LED, symbol Device:LED
- added IC1: LM393DR, digikey-footprints:SOIC-8_W3.9mm, symbol dk_Linear-Comparators:LM393DR
- added Q1: BS170, digikey-footprints:TO-92-3, symbol dk_Transistors-FETs-MOSFETs-Single:BS170
- added R1, R2, R3, R4, R5: R, symbol Device:R
- added Z1: 1N4733A, Diode_THT:D_DO-41_SOD81_P10.16mm_Horizontal, symbol Diode:1N47xxA
Connections:
- net at BT1.1 (+), BT2.1 (+): now also F1.2, IC1.6 (2IN-), R1.1, R2.1, R4.1, R5.1
- net GND: now reaches BT1.2 (-), BT2.2 (-)
- net GND: now also IC1.4 (GND), IC1.5 (2IN+), Q1.3 (S), R3.2, Z1.2 (A); no longer J1.2 (Pin_2)
- new net: D1.1 (K), J1.2 (Pin_2), Q1.1 (D)
- new net: IC1.2, R1.2, Z1.1 (K)
- new net: IC1.3, R2.2, R3.1
- new net: IC1.1 (1OUT), Q1.2 (G), R4.2
- new net: D1.2 (A), R5.2
Other:
- note added: "Load"
- moved on the sheet: BT1, BT2, F1, H1, H2, H3, H4, J1

Commit message: minor
Parts:
- D1: footprint (none) -> LED_SMD:LED_1206_3216Metric_Pad1.42x1.75mm_HandSolder
- IC1: footprint digikey-footprints:SOIC-8_W3.9mm -> Package_SO:SOIC-8_3.9x4.9mm_P1.27mm
- Q1: footprint digikey-footprints:TO-92-3 -> Package_TO_SOT_THT:TO-92_Inline_Wide
- R1, R2, R3, R4, R5: footprint (none) -> Resistor_SMD:R_1206_3216Metric_Pad1.42x1.75mm_HandSolder
Changed lines of the file:
@@
 F 0 "R1" H 3920 3646 50  0000 L CNN
 F 1 "R" H 3920 3555 50  0000 L CNN
-F 2 "" V 3780 3600 50  0001 C CNN
+F 2 "Resistor_SMD:R_1206_3216Metric_Pad1.42x1.75mm_HandSolder" V 3780 3600 50  0001 C CNN
 F 3 "~" H 3850 3600 50  0001 C CNN
 	1    3850 3600
@@
 F 0 "R2" H 4470 3646 50  0000 L CNN
 F 1 "R" H 4470 3555 50  0000 L CNN
-F 2 "" V 4330 3600 50  0001 C CNN
+F 2 "Resistor_SMD:R_1206_3216Metric_Pad1.42x1.75mm_HandSolder" V 4330 3600 50  0001 C CNN
 F 3 "~" H 4400 3600 50  0001 C CNN
 	1    4400 3600
@@
 F 0 "R4" H 5920 3646 50  0000 L CNN
 F 1 "R" H 5920 3555 50  0000 L CNN
-F 2 "" V 5780 3600 50  0001 C CNN
+F 2 "Resistor_SMD:R_1206_3216Metric_Pad1.42x1.75mm_HandSolder" V 5780 3600 50  0001 C CNN
 F 3 "~" H 5850 3600 50  0001 C CNN
 	1    5850 3600
@@
 F 0 "R5" H 6420 3646 50  0000 L CNN
 F 1 "R" H 6420 3555 50  0000 L CNN
-F 2 "" V 6280 3600 50  0001 C CNN
+F 2 "Resistor_SMD:R_1206_3216Metric_Pad1.42x1.75mm_HandSolder" V 6280 3600 50  0001 C CNN
 F 3 "~" H 6350 3600 50  0001 C CNN
 	1    6350 3600
@@
 F 0 "R3" H 4470 4696 50  0000 L CNN
 F 1 "R" H 4470 4605 50  0000 L CNN
-F 2 "" V 4330 4650 50  0001 C CNN
+F 2 "Resistor_SMD:R_1206_3216Metric_Pad1.42x1.75mm_HandSolder" V 4330 4650 50  0001 C CNN
 F 3 "~" H 4400 4650 50  0001 C CNN
 	1    4400 4650
@@
 F 0 "IC1" H 5150 4450 60  0000 L CNN
 F 1 "LM393DR" H 5150 4050 60  0000 L CNN
-F 2 "digikey-footprints:SOIC-8_W3.9mm" H 5150 4450 60  0001 L CNN
+F 2 "Package_SO:SOIC-8_3.9x4.9mm_P1.27mm" H 5150 4450 60  0001 L CNN
 F 3 "http://www.ti.com/lit/ds/symlink/lm193.pdf" H 5150 4550 60  0001 L CNN
 F 4 "296-1015-1-ND" H 5150 4650 60  0001 L CNN "Digi-Key_PN"
@@
 F 0 "Q1" H 6458 4653 60  0000 L CNN
 F 1 "BS170" H 6458 4547 60  0000 L CNN
-F 2 "digikey-footprints:TO-92-3" H 6550 4800 60  0001 L CNN
+F 2 "Package_TO_SOT_THT:TO-92_Inline_Wide" H 6550 4800 60  0001 L CNN
 F 3 "https://www.onsemi.com/pub/Collateral/BS170-D.PDF" H 6550 4900 60  0001 L CNN
 F 4 "BS170-ND" H 6550 5000 60  0001 L CNN "Digi-Key_PN"
@@
 F 0 "D1" V 6388 3883 50  0000 R CNN
 F 1 "LED" V 6297 3883 50  0000 R CNN
-F 2 "" H 6350 4000 50  0001 C CNN
+F 2 "LED_SMD:LED_1206_3216Metric_Pad1.42x1.75mm_HandSolder" H 6350 4000 50  0001 C CNN
 F 3 "~" H 6350 4000 50  0001 C CNN
 	1    6350 4000
@@
 $EndComp
 $Comp
-L power:GND #PWR?
+L power:GND #PWR0101
 U 1 1 5C971CEF
 P 5250 2850
-F 0 "#PWR?" H 5250 2600 50  0001 C CNN
+F 0 "#PWR0101" H 5250 2600 50  0001 C CNN
 F 1 "GND" H 5255 2677 50  0000 C CNN
 F 2 "" H 5250 2850 50  0001 C CNN
@@
 F 0 "IC1" H 5900 2800 60  0000 L CNN
 F 1 "LM393DR" H 5900 2400 60  0000 L CNN
-F 2 "digikey-footprints:SOIC-8_W3.9mm" H 5900 2800 60  0001 L CNN
+F 2 "Package_SO:SOIC-8_3.9x4.9mm_P1.27mm" H 5900 2800 60  0001 L CNN
 F 3 "http://www.ti.com/lit/ds/symlink/lm193.pdf" H 5900 2900 60  0001 L CNN
 F 4 "296-1015-1-ND" H 5900 3000 60  0001 L CNN "Digi-Key_PN"
@@
 $EndComp
 $Comp
-L power:GND #PWR?
+L power:GND #PWR0102
 U 1 1 5C975595
 P 3850 5000
-F 0 "#PWR?" H 3850 4750 50  0001 C CNN
+F 0 "#PWR0102" H 3850 4750 50  0001 C CNN
 F 1 "GND" H 3855 4827 50  0000 C CNN
 F 2 "" H 3850 5000 50  0001 C CNN
